File: hardware/PUTM_EV_PDMv2_PLAN_B_2024.kicad_sch (KiCad schematic)
At the start: 19 parts, among them J2 74650073R, J5 UMPT-08-01-L-RA-WT-P-TR, J8 UMPT-08-01-L-RA-WT-P-TR

Commit message: Version_after_fix2
Parts:
- FAN_1, FAN_2, FBOX_1, INVERTER_1, INVERTER_2, PC_2, PC_3, PC_4, PUMP_1, PUMP_2, SDC/ASMS_1: value ~ -> 2A
- J2: Mouser Url (none) -> https://eu.mouser.com/ProductDetail/Wurth-Elektronik/746500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
- PC_1: value 1 -> 2A
